File: mainboard-v05/Burn_Wires.kicad_sch (KiCad schematic)
At the start: 22 parts, among them Q20 NDS8434, Q21 NDS8434, Q4 IRLML2803, Q5 IRLML2803, Q6 MMBT2222AT, U16 PE014006

Commit message: Bumped schematic version to v05d. Changed parity warning priority
Parts:
- Q20, Q21: Field7 (none) -> NDS8434; Field8 (none) -> SO-8 ON Semiconductor
Changed lines of the file:
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@@
     )
   )
-  (symbol (lib_name "NDS8434_3") (lib_id "mainboard:NDS8434") (at 190.5 38.1 0) (unit 1)
+  (symbol (lib_id "mainboard:NDS8434") (at 190.5 38.1 0) (unit 1)
     (in_bom yes) (on_board yes) (dnp no)
     (property "Reference" "Q20" (at 182.88 26.67 0)
@@
       (effects (font (size 1.27 1.27)) (justify left bottom) hide)
     )
+    (property "Field7" "NDS8434" (at 190.5 38.1 0)
+      (effects (font (size 1.27 1.27)) (justify left bottom) hide)
+    )
+    (property "Field8" "SO-8 ON Semiconductor" (at 190.5 38.1 0)
+      (effects (font (size 1.27 1.27)) (justify left bottom) hide)
+    )
     (pin "1")
     (pin "2")
@@
     )
   )
-  (symbol (lib_name "NDS8434_4") (lib_id "mainboard:NDS8434") (at 190.5 62.23 0) (unit 1)
+  (symbol (lib_name "NDS8434_3") (lib_id "mainboard:NDS8434") (at 190.5 62.23 0) (unit 1)
     (in_bom yes) (on_board yes) (dnp no)
     (property "Reference" "Q21" (at 182.88 74.93 0)
@@
       (effects (font (size 1.27 1.27)) hide)
     )
+    (property "Field7" "NDS8434" (at 190.5 62.23 0)
+      (effects (font (size 1.27 1.27)) (justify left bottom) hide)
+    )
+    (property "Field8" "SO-8 ON Semiconductor" (at 190.5 62.23 0)
+      (effects (font (size 1.27 1.27)) (justify left bottom) hide)
+    )
     (pin "1")
