File: mainboard-v05/Power.kicad_sch (KiCad schematic)
At the start: 70 parts, among them J14 Conn_01x06, Q1 IRLML2803, Q2 MBT2222ADW1T1, Q22 NDS8434, Q3 MBT2222ADW1T1, U17 BQ25883RGER, U21 TPS7A4501DCQT, U4 ADM1176-1ARMZ-R7, U5 TPS54226PWPRPWP14_2P31X2P46-L, U6 LTC4121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

Commit message: Bumped schematic version to v05d. Changed parity warning priority
Parts:
- Q22: Field7 (none) -> NDS8434; Field8 (none) -> SO-8 ON Semiconductor
Changed lines of the file:
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@@
     )
   )
-  (symbol (lib_name "NDS8434_2") (lib_id "mainboard:NDS8434") (at 251.46 43.18 0) (unit 1)
+  (symbol (lib_id "mainboard:NDS8434") (at 251.46 43.18 0) (unit 1)
     (in_bom yes) (on_board yes) (dnp no)
     (property "Reference" "Q22" (at 250.19 31.75 0)
@@
       (effects (font (size 1.27 1.27)) hide)
     )
+    (property "Field7" "NDS8434" (at 251.46 43.18 0)
+      (effects (font (size 1.27 1.27)) (justify left bottom) hide)
+    )
+    (property "Field8" "SO-8 ON Semiconductor" (at 251.46 43.18 0)
+      (effects (font (size 1.27 1.27)) (justify left bottom) hide)
+    )
     (pin "1")
